File: Haish.kicad_pcb (KiCad board)
At the start: 2 copper layers, 262 x 77 mm, 93 parts, among them U1 ProMicro

Commit message: rampung.
Routing:
- net KOLOM0: track 0.00 -> 334.6 mm
- net KOLOM1: track 0.00 -> 315.1 mm
- net KOLOM2: track 0.00 -> 293.2 mm
- net BARIS3: track 0.00 -> 290.4 mm
- net KOLOM3: track 0.00 -> 271.6 mm
- net BARIS2: track 0.00 -> 258.2 mm
- net BARIS1: track 0.00 -> 245.4 mm
- net BARIS0: track 0.00 -> 238.5 mm
- net KOLOM4: track 0.00 -> 228.5 mm
- net KOLOM5: track 0.00 -> 226.5 mm
- net KOLOM6: track 0.00 -> 186.9 mm
- net KOLOM7: track 0.00 -> 185.6 mm
- net KOLOM8: track 0.00 -> 157.8 mm, vias 0 -> 1
- net KOLOM9: track 0.00 -> 138.9 mm, vias 0 -> 1
- net KOLOMA: track 0.00 -> 118.8 mm, vias 0 -> 1
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