File: Haish.sch (KiCad schematic (older format))
At the start: 93 parts, among them K1 KEYSW, K10 KEYSW, K11 KEYSW, K12 KEYSW, K13 KEYSW, K14 KEYSW, K15 KEYSW, K16 KEYSW, K17 KEYSW, K18 KEYSW, K19 KEYSW, K2 KEYSW, K20 KEYSW, K21 KEYSW, K22 KEYSW, K23 KEYSW, K24 KEYSW, K25 KEYSW, K26 KEYSW, K27 KEYSW, K28 KEYSW, K29 KEYSW, K3 KEYSW, K30 KEYSW, K31 KEYSW, K32 KEYSW, K33 KEYSW, K34 KEYSW, K35 KEYSW, K36 KEYSW, K37 KEYSW, K38 KEYSW, K39 KEYSW, K4 KEYSW, K40 KEYSW, K41 KEYSW, K42 KEYSW, K43 KEYSW, K44 KEYSW, K45 KEYSW, K5 KEYSW, K6 KEYSW, K7 KEYSW, K8 KEYSW, K9 KEYSW, U1 ProMicro

Commit message: hhmm...' '
Parts:
- renumbered K?1 to K0
Changed lines of the file:
@@
 $EndDescr
 $Comp
-L keyboard_parts:KEYSW K?1
+L keyboard_parts:KEYSW K0
 U 1 1 5DE1411D
 P 1900 1000
-F 0 "K?1" H 1900 1233 60  0000 C CNN
+F 0 "K0" H 1900 1233 60  0000 C CNN
 F 1 "KEYSW" H 1900 900 60  0001 C CNN
 F 2 "Keebio-Parts:MX_PCB_100H" H 1900 1000 60  0001 C CNN

Commit message: hhmm...' '
Parts:
- K-0-B1: renamed from K42; footprint Keebio-Parts:MX_PCB_100H -> Keebio-Parts:MX_PCB_125H
- K-1-0: renamed from K1; footprint Keebio-Parts:MX_PCB_100H -> Keebio-Parts:MX_PCB_125H
- K-2-0: renamed from K2; footprint Keebio-Parts:MX_PCB_100H -> Keebio-Parts:MX_PCB_175H
- K-3-0: renamed from K3; footprint Keebio-Parts:MX_PCB_100H -> Keebio-Parts:MX_PCB_125H
- K-3-2: renamed from K11; footprint Keebio-Parts:MX_PCB_100H -> Keebio-Parts:MX_PCB_125H
- K-3-3: renamed from K15; footprint Keebio-Parts:MX_PCB_100H -> Keebio-Parts:MX_PCB_225H
- K-3-7: renamed from K29; footprint Keebio-Parts:MX_PCB_100H -> Keebio-Parts:MX_PCB_275H
- K-3-8: renamed from K33; footprint Keebio-Parts:MX_PCB_100H -> Keebio-Parts:MX_PCB_125H
- renumbered D1 to D-0-0, D5 to D-0-1, D9 to D-0-2, D13 to D-0-3, D17 to D-0-4, D20 to D-0-5, D24 to D-0-6, D27 to D-0-7, D31 to D-0-8, D35 to D-0-9, D39 to D-0-A1, D43 to D-0-B1, D2 to D-1-0, D6 to D-1-1, D10 to D-1-2, D14 to D-1-3, D18 to D-1-4, D21 to D-1-5, D25 to D-1-6, D28 to D-1-7, D32 to D-1-8, D36 to D-1-9, D40 to D-1-A1, D44 to D-1-B1, D3 to D-2-0, D7 to D-2-1, D11 to D-2-2, D15 to D-2-3, D19 to D-2-4, D22 to D-2-5, D26 to D-2-6, D29 to D-2-7, D33 to D-2-8, D37 to D-2-9, D41 to D-2-A1, D45 to D-2-B1, D4 to D-3-0, D8 to D-3-1, D12 to D-3-2, D16 to D-3-3, D23 to D-3-5, D30 to D-3-7, D34 to D-3-8, D38 to D-3-9, D42 to D-3-A1, D46 to D-3-B1, K0 to K-0-0, K4 to K-0-1, K8 to K-0-2, K12 to K-0-3, K16 to K-0-4, K19 to K-0-5, K23 to K-0-6, K26 to K-0-7, K30 to K-0-8, K34 to K-0-9, K38 to K-0-A1, K5 to K-1-1, K9 to K-1-2, K13 to K-1-3, K17 to K-1-4, K20 to K-1-5, K24 to K-1-6, K27 to K-1-7, K31 to K-1-8, K35 to K-1-9, K39 to K-1-A1, K43 to K-1-B1, K6 to K-2-1, K10 to K-2-2, K14 to K-2-3, K18 to K-2-4, K21 to K-2-5, K25 to K-2-6, K28 to K-2-7, K32 to K-2-8, K36 to K-2-9, K40 to K-2-A1, K44 to K-2-B1, K7 to K-3-1, K22 to K-3-5, K37 to K-3-9, K41 to K-3-A1, K45 to K-3-B1
